File: semi.kicad_pcb (KiCad board)
At the start: 2 copper layers, 234.9 x 77.8 mm, 121 parts, among them SW1 SW_Push, U1 SRV05-4, U2 ATmega32U4-AU, Y1 Resonator_Small

Commit message: Updated PCB & Fixes
Removed nonfunctional screw holes
Added 32u4-MU footprint
Updated PCB files to KiCad 6
Updated production files to match
Parts:
- removed H1, H2, H3, H4: MountingHole_Pad, MountingHole:MountingHole_2.2mm_M2_Pad
- added U3: ATmega32U4-M, Package_DFN_QFN:QFN-44-1EP_7x7mm_P0.5mm_EP5.2x5.2mm, B.Cu at (29.8, 39.9)
Connections:
- USB1 pad 3: Net-(USB1-Pad3) -> unconnected-(USB1-Pad3)
- USB1 pad 9: Net-(USB1-Pad9) -> unconnected-(USB1-Pad9)
Routing:
- net +5V: track 116.3 -> 131.7 mm
- net col1: track 83.0 -> 76.4 mm, vias 0 -> 1
- net col3: track 69.0 -> 72.1 mm
- net Net-(U2-Pad10): track 0.00 -> 3.04 mm
- net Net-(R1-Pad2): track 15.8 -> 18.8 mm
- net col2: track 76.2 -> 79.2 mm
- net Net-(U2-Pad12): track 0.00 -> 2.98 mm
- net Net-(U2-Pad11): track 0.00 -> 2.98 mm
- net Net-(U2-Pad1): track 0.00 -> 2.98 mm
- net Net-(R6-Pad2): track 2.06 -> 5.05 mm
- net col4: track 115.0 -> 117.9 mm
- net col10: track 252.9 -> 255.7 mm
- net row2: track 225.3 -> 228.0 mm
- net Net-(U2-Pad9): track 0.00 -> 2.74 mm
- net D-: track 24.8 -> 27.6 mm
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Other:
- net class Default removed
